Commit message: Dynamixel fix to vel control

File: open_manipulator_x_description/urdf/open_manipulator_x.ros2_control.xacro (robot description, xacro)
@@ -5,10 +5,10 @@
       <hardware>
         <plugin>dynamixel_hardware/DynamixelHardware</plugin>
-        <param name="usb_port">/dev/ttyUSB0</param>
+        <param name="usb_port">/dev/ttyUSB_DYNAMIXE</param>
         <param name="baud_rate">1000000</param>
         <!-- <param name="use_dummy">true</param> -->
       </hardware>
       <joint name="joint1">
-        <param name="id">11</param>
+        <param name="id">1</param>
         <command_interface name="position"/>
         <command_interface name="velocity"/>
@@ -18,5 +18,5 @@
       </joint>
       <joint name="joint2">
-        <param name="id">12</param>
+        <param name="id">2</param>
         <command_interface name="position"/>
         <command_interface name="velocity"/>
@@ -26,5 +26,5 @@
       </joint>
       <joint name="joint3">
-        <param name="id">13</param>
+        <param name="id">3</param>
         <command_interface name="position"/>
         <command_interface name="velocity"/>
@@ -34,5 +34,5 @@
       </joint>
       <joint name="joint4">
-        <param name="id">14</param>
+        <param name="id">4</param>
         <command_interface name="position"/>
         <command_interface name="velocity"/>
@@ -41,5 +41,5 @@
         <state_interface name="effort"/>
       </joint>
-      <joint name="gripper">
+      <!-- <joint name="gripper">
         <param name="id">15</param>
         <command_interface name="position"/>
@@ -48,5 +48,5 @@
         <state_interface name="velocity"/>
         <state_interface name="effort"/>
-      </joint>
+      </joint> -->
     </ros2_control>
   </xacro:macro>
